Commit message: Finished Project

File: urdf_test/src/myrobot_description/urdf/gazebo (copy).xacro (robot description, xacro)
@@ -9,4 +9,12 @@
         <static>true</static>
     </gazebo>
+    <gazebo reference="base_Link__gG_Rechts">
+	<mu1>150</mu1>
+    	<mu2>50</mu2>
+    </gazebo>
+    <gazebo reference="gG_Rechts__gG_Links">
+	<mu1>150</mu1>
+    	<mu2>50</mu2>
+    </gazebo>
     <gazebo reference="gG_Links__unterSchwinge">
 	<disableFixedJointLumping>true</disableFixedJointLumping>
@@ -15,6 +23,24 @@
 	<disableFixedJointLumping>true</disableFixedJointLumping>
     </gazebo>
+    <gazebo reference="mG_Links__mG_Rechts">
+	<mu1>180</mu1>
+    	<mu2>70</mu2>
+    </gazebo>
+    <gazebo reference="mG_Rechts__oberSchwinge">
+	<mu1>100</mu1>
+    	<mu2>40</mu2>
+    </gazebo>
     <gazebo reference="oberSchwinge__kG_Rechts">
 	<disableFixedJointLumping>true</disableFixedJointLumping>
     </gazebo>
+    <gazebo reference="kG_Rechts__kG_Links">
+	<mu1>40</mu1>
+    	<mu2>10</mu2>
+    </gazebo>
+    <gazebo reference="kG_Links__endEffektor">
+	<mu1>1000</mu1>
+    	<mu2>1000</mu2>
+	<kp>1000</kp>
+    	<kd>1000</kd>
+    </gazebo>
 </robot>

File: urdf_test/src/myrobot_description/urdf/links_joints.xacro (robot description, xacro)
@@ -55,5 +55,5 @@
 		<joint name="${name}" type="revolute">
 			<axis xyz="${axis_xyz}" />
-			<limit effort="${effort_limit}" lower="-3.14" upper="3.14" velocity="0.1"/>
+			<limit effort="${effort_limit}" lower="-3.14" upper="3.14" velocity="2"/>
 			<origin xyz="${origin_xyz}" rpy="${origin_rpy}" />
 			<parent link="${parent}"/>

File: urdf_test/src/myrobot_description/urdf/robot_parameters.xacro (robot description, xacro)
@@ -20,5 +20,5 @@
 	<xacro:property name="mG_length" value="0.152" />
 	<xacro:property name="mG_radius" value="0.065" />
-	<xacro:property name="mG_effort" value="200" />
+	<xacro:property name="mG_effort" value="300" />
 	<xacro:property name="mG_mass" value="5.269" />
 	<!-- properties of the small motors/links -->
